Commit message: feat: walk work

File: resources/robots/bruce/bruce_bak.urdf (robot description, URDF)
Before this commit: robot bruce, 17 links, 16 joints
Links:
- link hip_pitch_link_l: geometry collision mesh filename=/home/bigeast/pbrs-humanoid/resources/robots/bruce/meshes_v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; visual mesh filename=/home/bigeast/pbrs-humanoid/resources/robots/bruce/meshes_v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
- link hip_pitch_link_r: geometry collision mesh filename=/home/bigeast/pbrs-humanoid/resources/robots/bruce/meshes_v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; visual mesh filename=/home/bigeast/pbrs-humanoid/resources/robots/bruce/meshes_v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
