Commit message: feat: work!

File: resources/robots/bruce/bruce.urdf (robot description, URDF)
Before this commit: robot bruce, 17 links, 16 joints
Joints:
- joint ankle_pitch_l: limit lower=-3.1415 upper=3.1415 effort=1000 velocity=1000 -> lower=-1.0 upper=1.0 effort=1000 velocity=1000
- joint ankle_pitch_r: limit lower=-3.1415 upper=3.1415 effort=1000 velocity=1000 -> lower=-1.0 upper=1.0 effort=1000 velocity=1000

Commit message: feat: stand work in more inertia!

File: resources/robots/bruce/bruce.urdf (robot description, URDF)
Before this commit: robot bruce, 17 links, 16 joints
Joints:
- joint elbow_pitch_l: type fixed -> revolute
- joint elbow_pitch_r: type fixed -> revolute
- joint shoulder_pitch_l: type fixed -> revolute
- joint shoulder_pitch_r: type fixed -> revolute
- joint shoulder_roll_l: type fixed -> revolute
- joint shoulder_roll_r: type fixed -> revolute
